File: circuitry/System Schematic.sch (EAGLE design)
At the start: 16 parts

Commit message: Update schematic to most recent hardware prototype
Parts:
- removed R7: RESISTOR_0603_1K, roboGech_devices:RESISTOR_0603_1K
- D1, D2, D3, D4: value LED_0603_WHITE -> LED_0603_RED; device roboGech_devices:LED_0603_WHITE -> HyTechDevices:LED_0603_RED
Connections:
- removed net N$18: LED1.BA, R7.2
- removed net RGB_BLUE: ESP32_CAM.IO16, R7.1
- new net BUILTIN_FLASH: ESP32_CAM.IO4
- new net N$12: U$3.GND
- net GND: now also LED1.BA; no longer U$3.GND
- net RGB_GREEN: now also ESP32_CAM.IO16; no longer ESP32_CAM.IO4
Changed lines of the file:
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@@
 <part name="P4" library="roboGech_devices" library_urn="urn:adsk.eagle:library:35088295" deviceset="GND" device=""/>
 <part name="P5" library="roboGech_devices" library_urn="urn:adsk.eagle:library:35088295" deviceset="GND" device=""/>
-<part name="U$3" library="roboGech_devices" library_urn="urn:adsk.eagle:library:35088295" deviceset="ULN2003_DRIVER" device="" package3d_urn="urn:adsk.eagle:package:35088325/1"/>
+<part name="U$3" library="roboGech_devices" deviceset="ULN2003_DRIVER" device=""/>
 <part name="U$4" library="roboGech_devices" library_urn="urn:adsk.eagle:library:35088295" deviceset="28BYJ-48" device="" package3d_urn="urn:adsk.eagle:package:35088324/1"/>
-<part name="P6" library="roboGech_devices" library_urn="urn:adsk.eagle:library:35088295" deviceset="GND" device=""/>
 <part name="P7" library="roboGech_devices" library_urn="urn:adsk.eagle:library:35088295" deviceset="+5V" device=""/>
 <part name="P8" library="roboGech_devices" library_urn="urn:adsk.eagle:library:35088295" deviceset="+5V" device=""/>
-<part name="D1" library="roboGech_devices" library_urn="urn:adsk.eagle:library:35088295" deviceset="LED_?_*" device="0603" package3d_urn="urn:adsk.eagle:package:35088319/1" technology="WHITE"/>
-<part name="D2" library="roboGech_devices" library_urn="urn:adsk.eagle:library:35088295" deviceset="LED_?_*" device="0603" package3d_urn="urn:adsk.eagle:package:35088319/1" technology="WHITE"/>
-<part name="D3" library="roboGech_devices" library_urn="urn:adsk.eagle:library:35088295" deviceset="LED_?_*" device="0603" package3d_urn="urn:adsk.eagle:package:35088319/1" technology="WHITE"/>
-<part name="D4" library="roboGech_devices" library_urn="urn:adsk.eagle:library:35088295" deviceset="LED_?_*" device="0603" package3d_urn="urn:adsk.eagle:package:35088319/1" technology="WHITE"/>
+<part name="D1" library="HyTechDevices" deviceset="LED_?_*" device="0603" technology="RED" value="LED_0603_RED"/>
+<part name="D2" library="HyTechDevices" deviceset="LED_?_*" device="0603" technology="RED" value="LED_0603_RED"/>
+<part name="D3" library="HyTechDevices" deviceset="LED_?_*" device="0603" technology="RED" value="LED_0603_RED"/>
+<part name="D4" library="HyTechDevices" deviceset="LED_?_*" device="0603" technology="RED" value="LED_0603_RED"/>
 <part name="R1" library="roboGech_devices" library_urn="urn:adsk.eagle:library:35088295" deviceset="RESISTOR_?_*" device="0603" package3d_urn="urn:adsk.eagle:package:35088322/1" technology="1K"/>
 <part name="R2" library="roboGech_devices" library_urn="urn:adsk.eagle:library:35088295" deviceset="RESISTOR_?_*" device="0603" package3d_urn="urn:adsk.eagle:package:35088322/1" technology="1K"/>
@@
 <part name="R5" library="roboGech_devices" library_urn="urn:adsk.eagle:library:35088295" deviceset="RESISTOR_?_*" device="0603" package3d_urn="urn:adsk.eagle:package:35088322/1" technology="1K"/>
 <part name="R6" library="roboGech_devices" library_urn="urn:adsk.eagle:library:35088295" deviceset="RESISTOR_?_*" device="0603" package3d_urn="urn:adsk.eagle:package:35088322/1" technology="1K"/>
-<part name="R7" library="roboGech_devices" library_urn="urn:adsk.eagle:library:35088295" deviceset="RESISTOR_?_*" device="0603" package3d_urn="urn:adsk.eagle:package:35088322/1" technology="1K"/>
+<part name="P6" library="roboGech_devices" deviceset="GND" device=""/>
 </parts>
 <sheets>
@@
 <attribute name="NAME" x="49.53" y="144.78" size="1.778" layer="95"/>
 </instance>
-<instance part="P1" gate="1" x="215.9" y="161.29" smashed="yes">
-<attribute name="VALUE" x="215.9" y="160.02" size="1.27" layer="96" align="top-center"/>
+<instance part="P1" gate="1" x="215.9" y="151.13" smashed="yes">
+<attribute name="VALUE" x="215.9" y="149.86" size="1.27" layer="96" align="top-center"/>
 </instance>
 <instance part="P3" gate="1" x="95.25" y="92.71" smashed="yes">
@@
 <attribute name="VALUE" x="235.331" y="88.9" size="1.778" layer="96"/>
 </instance>
-<instance part="P6" gate="1" x="153.67" y="83.82" smashed="yes">
-<attribute name="VALUE" x="153.67" y="82.55" size="1.27" layer="96" align="top-center"/>
-</instance>
 <instance part="P7" gate="1" x="139.7" y="110.49" smashed="yes">
 <attribute name="VALUE" x="139.7" y="113.03" size="1.27" layer="96" align="bottom-center"/>
@@
 <attribute name="RESISTANCE" x="187.96" y="172.72" size="1.27" layer="96" align="top-center"/>
 </instance>
-<instance part="R7" gate="G$1" x="189.23" y="168.91" smashed="yes">
-<attribute name="NAME" x="187.96" y="170.18" size="1.27" layer="95" align="bottom-center"/>
-<attribute name="RESISTANCE" x="187.96" y="167.64" size="1.27" layer="96" align="top-center"/>
+<instance part="P6" gate="1" x="187.96" y="76.2" smashed="yes">
+<attribute name="VALUE" x="187.96" y="74.93" size="1.27" layer="96" align="top-center"/>
 </instance>
 </instances>
@@
 <pinref part="LED1" gate="G$1" pin="RC"/>
 <wire x1="215.9" y1="173.99" x2="215.9" y2="168.91" width="0.1524" layer="91"/>
-<wire x1="215.9" y1="168.91" x2="215.9" y2="163.83" width="0.1524" layer="91"/>
+<wire x1="215.9" y1="168.91" x2="215.9" y2="157.48" width="0.1524" layer="91"/>
+<wire x1="215.9" y1="157.48" x2="215.9" y2="153.67" width="0.1524" layer="91"/>
 <wire x1="200.66" y1="179.07" x2="215.9" y2="179.07" width="0.1524" layer="91"/>
 <pinref part="LED1" gate="G$1" pin="GC"/>
@@
 <wire x1="200.66" y1="168.91" x2="215.9" y2="168.91" width="0.1524" layer="91"/>
 <junction x="215.9" y="168.91"/>
+<pinref part="LED1" gate="G$1" pin="BA"/>
+<wire x1="195.58" y1="168.91" x2="187.96" y2="168.91" width="0.1524" layer="91"/>
+<wire x1="187.96" y1="168.91" x2="187.96" y2="157.48" width="0.1524" layer="91"/>
+<wire x1="187.96" y1="157.48" x2="215.9" y2="157.48" width="0.1524" layer="91"/>
+<junction x="215.9" y="157.48"/>
 </segment>
 <segment>
@@
 <wire x1="22.86" y1="138.43" x2="22.86" y2="120.65" width="0.1524" layer="91"/>
 <pinref part="P5" gate="1" pin="GND"/>
-</segment>
-<segment>
-<pinref part="U$3" gate="G$1" pin="GND"/>
-<wire x1="158.75" y1="88.9" x2="153.67" y2="88.9" width="0.1524" layer="91"/>
-<wire x1="153.67" y1="88.9" x2="153.67" y2="86.36" width="0.1524" layer="91"/>
-<pinref part="P6" gate="1" pin="GND"/>
 </segment>
 <segment>
@@
 <net name="N$7" class="0">
 <segment>
+<wire x1="139.7" y1="88.9" x2="139.7" y2="107.95" width="0.1524" layer="91"/>
+<pinref part="P7" gate="1" pin="+5V"/>
 <pinref part="U$3" gate="G$1" pin="5V"/>
-<wire x1="158.75" y1="91.44" x2="139.7" y2="91.44" width="0.1524" layer="91"/>
-<wire x1="139.7" y1="91.44" x2="139.7" y2="107.95" width="0.1524" layer="91"/>
-<pinref part="P7" gate="1" pin="+5V"/>
+<wire x1="139.7" y1="88.9" x2="158.75" y2="88.9" width="0.1524" layer="91"/>
 </segment>
 </net>
@@
 <net name="RGB_GREEN" class="0">
 <segment>
-<pinref part="ESP32_CAM" gate="G$1" pin="IO4"/>
-<wire x1="44.45" y1="123.19" x2="39.37" y2="123.19" width="0.1524" layer="91"/>
-<label x="39.116" y="123.19" size="1.27" layer="95" font="vector" rot="MR0" xref="yes"/>
-</segment>
-<segment>
 <pinref part="R6" gate="G$1" pin="1"/>
 <wire x1="184.15" y1="173.99" x2="180.34" y2="173.99" width="0.1524" layer="91"/>
 <label x="180.34" y="173.99" size="1.27" layer="95" font="vector" rot="MR0" xref="yes"/>
 </segment>
-</net>
-<net name="RGB_BLUE" class="0">
 <segment>
 <pinref part="ESP32_CAM" gate="G$1" pin="IO16"/>
@@
 <label x="81.28" y="138.43" size="1.27" layer="95" font="vector" xref="yes"/>
 </segment>
-<segment>
-<pinref part="R7" gate="G$1" pin="1"/>
-<wire x1="184.15" y1="168.91" x2="179.07" y2="168.91" width="0.1524" layer="91"/>
-<label x="179.07" y="168.91" size="1.27" layer="95" font="vector" rot="MR0" xref="yes"/>
-</segment>
 </net>
 <net name="N$16" class="0">
@@
 </segment>
 </net>
-<net name="N$18" class="0">
-<segment>
-<pinref part="R7" gate="G$1" pin="2"/>
-<pinref part="LED1" gate="G$1" pin="BA"/>
-<wire x1="191.77" y1="168.91" x2="195.58" y2="168.91" width="0.1524" layer="91"/>
-</segment>
-</net>
+<net name="N$12" class="0">
+<segment>
+<pinref part="U$3" gate="G$1" pin="GND"/>
+<wire x1="186.69" y1="88.9" x2="187.96" y2="88.9" width="0.1524" layer="91"/>
+<wire x1="187.96" y1="88.9" x2="187.96" y2="78.74" width="0.1524" layer="91"/>
+<pinref part="P6" gate="1" pin="GND"/>
+</segment>
+</net>
+<net name="BUILTIN_FLASH" class="0">
+<segment>
+<pinref part="ESP32_CAM" gate="G$1" pin="IO4"/>
+<wire x1="44.45" y1="123.19" x2="42.672" y2="123.19" width="0.1524" layer="91"/>
+<label x="42.418" y="123.19" size="1.27" layer="95" font="vector" rot="MR0" xref="yes"/>
+</segment>
+</net>
